Commit message: fix robot xacro file
fix robot xacro file so that it moves fluently when given /cmd_vel

File: my_robot/urdf/my_robot.xacro (robot description, xacro)
@@ -19,8 +19,8 @@
       />
     </inertial>
-    <collision name='collision'>
+   <collision name='chasis_collision'>
       <origin xyz="0 0 0" rpy=" 0 0 0"/>
       <geometry>
-        <box size=".6 .2 .1"/>
+        <box size=".4 .2 .1"/>
       </geometry>
     </collision>
@@ -28,29 +28,29 @@
       <origin xyz="0 0 0" rpy=" 0 0 0"/>
       <geometry>
-        <box size=".6 .2 .1"/>
+        <box size=".4 .2 .1"/>
       </geometry>
     </visual>
     <collision name='back_caster_collision'>
-      <origin xyz="-0.15 0 -0.1" rpy=" 0 0 0"/>
+      <origin xyz="-0.15 0 -0.05" rpy=" 0 0 0"/>
       <geometry>
-        <sphere radius="0.1"/>
+        <sphere radius="0.0499"/>
       </geometry>
     </collision>
     <visual name='back_caster_visual'>
-      <origin xyz="-0.15 0 -0.1" rpy=" 0 0 0"/>
+      <origin xyz="-0.15 0 -0.05" rpy=" 0 0 0"/>
       <geometry>
-        <sphere radius="0.1"/>
+        <sphere radius="0.05"/>
       </geometry>
     </visual>
     <collision name='front_caster_collision'>
-      <origin xyz="0.15 0 -0.1" rpy=" 0 0 0"/>
+      <origin xyz="0.15 0 -0.05" rpy=" 0 0 0"/>
       <geometry>
-        <sphere radius="0.1"/>
+        <sphere radius="0.0499"/>
       </geometry>
     </collision>
     <visual name='front_caster_visual'>
-      <origin xyz="0.15 0 -0.1" rpy=" 0 0 0"/>
+      <origin xyz="0.15 0 -0.05" rpy=" 0 0 0"/>
       <geometry>
-        <sphere radius="0.1"/>
+        <sphere radius="0.05"/>
       </geometry>
     </visual>
@@ -70,5 +70,5 @@
       <origin xyz="0 0 0" rpy=" 0 1.5707 1.5707"/>
       <geometry>
-        <cylinder radius=".2" length="0.05"/>
+        <cylinder radius=".1" length="0.05"/>
       </geometry>
     </collision>
@@ -76,5 +76,5 @@
       <origin xyz="0 0 0" rpy=" 0 1.5707 1.5707"/>
       <geometry>
-        <cylinder radius=".2" length="0.05"/>
+        <cylinder radius=".1" length="0.05"/>
       </geometry>
     </visual>
@@ -102,5 +102,5 @@
       <origin xyz="0 0 0" rpy=" 0 1.5707 1.5707"/>
       <geometry>
-        <cylinder radius=".2" length="0.05"/>
+        <cylinder radius=".1" length="0.05"/>
       </geometry>
     </collision>
@@ -108,5 +108,5 @@
       <origin xyz="0 0 0" rpy=" 0 1.5707 1.5707"/>
       <geometry>
-        <cylinder radius=".2" length="0.05"/>
+        <cylinder radius=".1" length="0.05"/>
       </geometry>
     </visual>
@@ -145,5 +145,5 @@
    </link>
    <joint type="fixed" name="camera_joint">
-     <origin xyz="0.3 0 0" rpy="0 0 0"/>
+     <origin xyz="0.2 0 0" rpy="0 0 0"/>
      <child link="camera"/>
      <parent link="chassis"/>
